File: cistercian_clock_kicad/cistercian_clock.kicad_sch (KiCad schematic)
At the start: 1 part, among them U1 ATmega328PB-A

Commit message: started code for clock cycles, updated schematics
Parts:
- added A1: Arduino_Nano_v2.x, Module:Arduino_Nano, symbol MCU_Module:Arduino_Nano_v2.x
Connections:
- net A0: now also A1.22 (A3)
- net A1: now also A1.15 (D12)
- net A2: now also A1.10 (D7)
- net A3: now also A1.5 (D2)
- net B0: now also A1.23 (A4)
- net B1: now also A1.16 (D13)
- net B2: now also A1.11 (D8)
- net B3: now also A1.6 (D3)
- net C0: now also A1.24 (A5)
- net C1: now also A1.19 (A0)
- net C2: now also A1.12 (D9)
- net C3: now also A1.7 (D4)
- net D0: now also A1.25 (A6)
- net D1: now also A1.20 (A1)
- net D2: now also A1.13 (D10)
- net D3: now also A1.8 (D5)
- net E0: now also A1.26 (A7)
- net E1: now also A1.21 (A2)
- net E2: now also A1.14 (D11)
- net E3: now also A1.9 (D6)
- net MID renamed F4
- net F4: now also A1.2 (D0/RX)
